Commit message: Perfected readme,Python invoked the MoveIt inverse kinematics interface.

File: install/cpp06_urdf/share/cpp06_urdf/urdf/xacro/car.urdf.xacro (robot description, xacro)
@@ -1,14 +1 @@
-<robot xmlns:xacro="http://www.ros.org/wiki/xacro" name="car">
-    <xacro:include filename="car_base.urdf.xacro"/>
-    <xacro:include filename="car_camera.urdf.xacro"/>
-    <xacro:include filename="car_laser.urdf.xacro"/>
-    <xacro:include filename="car_imu.urdf.xacro"/>
-    <xacro:include filename="car_caster.urdf.xacro"/>
-    <!-- <xacro:include filename="gazebo_control_plugin.xacro"/> -->
-    <xacro:include filename="gazebo_sensor_plugin.xacro"/>
-    <xacro:include filename="car_control.urdf.xacro"/>
-    <xacro:imu_xacro xyz="0 0 0.02" />
-    <!-- <xacro:gazebo_control_plugin /> -->
-    <xacro:gazebo_sensor_plugin />
-    <xacro:car_control />
-</robot>
+/home/wz/Desktop/ROS_ROBOT/src/cpp06_urdf/urdf/xacro/car.urdf.xacro

File: install/cpp06_urdf/share/cpp06_urdf/urdf/xacro/car_base.urdf.xacro (robot description, xacro)
@@ -1,98 +1 @@
-<?xml version="1.0"?>
-<robot xmlns:xacro="http://www.ros.org/wiki/xacro">
-    <xacro:include filename="$(find cpp06_urdf)/urdf/xacro/common_inertia.xacro"/>
-    <!-- 1.需要声明变量 -->
-    <xacro:property name="PI" value="3.1415927" />
-    <xacro:property name="car_length" value="0.2" />
-    <xacro:property name="car_width" value="0.12" />
-    <xacro:property name="car_height" value="0.07" />
-    <xacro:property name="wheel_radius" value="0.025" />
-    <xacro:property name="wheel_length" value="0.02" />
-    <!-- 轮胎关节偏移量 -->
-    <xacro:property name="wheel_joint_x" value="0.08" />
-    <xacro:property name="wheel_joint_y" value="${car_width / 2}" />
-    <xacro:property name="wheel_joint_z" value="${-(car_height / 2 + distance - wheel_radius)}" />
-    <!-- 离地间隙 -->
-    <xacro:property name="distance" value="0.015" />
-    <material name="yellow">
-        <color rgba="0.9 0.6 0.0 0.5"/>
-    </material>
-    <material name="black">
-        <color rgba="0.0 0.0 0.0 0.5"/>
-    </material>
-    <!-- 2.设置base_footprint -->
-    <link name="base_footprint">
-        <visual>
-            <geometry>
-                <sphere radius="0.001"/>
-            </geometry>
-        </visual>
-    </link>
-    <!-- 3.设置base_link -->
-    <link name="base_link">
-        <visual>
-            <geometry>
-                <box size="${car_length} ${car_width} ${car_height}"/>
-            </geometry>
-            <material name="yellow"/>
-        </visual>
-        <collision>
-             <geometry>
-                <box size="${car_length} ${car_width} ${car_height}"/>
-            </geometry>
-            <material name="yellow"/>
-        </collision>
-        <xacro:box_inertia m="1.0" d="${car_length}" w="${car_width}" h="${car_height}" />
-    </link>
-    <!-- 4.使用joint将二者相联 -->
-    <joint name="base_link2base_footprint" type="fixed">
-        <parent link="base_footprint"/>
-        <child link="base_link"/>
-        <origin xyz="0.0 0.0 ${car_height/2 + distance}"/>
-    </joint>
-    <!-- 5.定义车轮相关的宏 -->
-    <!-- 宏函数创建规则,封装通用代码（可被复用的代码），变的数据以参数的方式暴露出去 -->
-    <!-- link变量：name -->
-    <!-- joint变量：name child-link origin(x y z)-->
-    <xacro:macro name="wheel_func" params="link_name front_flag left_flag">
-        <link name="${link_name}">
-            <visual>
-                <geometry>
-                    <cylinder radius="${wheel_radius}" length="${wheel_length}"/>
-                </geometry>
-                <material name="black"/>
-                <origin rpy="${PI/2} 0.0 0.0"/>
-            </visual>
-            <collision>
-                <geometry>
-                    <cylinder radius="${wheel_radius}" length="${wheel_length}"/>
-                </geometry>
-                <material name="black"/>
-                <origin rpy="${PI/2} 0.0 0.0"/>
-            </collision>
-            <xacro:cylinder_inertia m="1.0" r="${wheel_radius}" h="${wheel_length}" />
-        </link>
-            <joint name="${link_name}2base_link" type="continuous">
-            <parent link="base_link"/>
-            <child link="${link_name}"/>
-            <origin xyz="${wheel_joint_x * front_flag} ${wheel_joint_y * left_flag} ${wheel_joint_z}"/>
-            <axis xyz="0 1 0"/>
-        </joint>
-        <gazebo reference="${link_name}">
-            <!-- 切向的摩擦系数 -->
-            <mu1 value="20.0" />
-            <!-- 法向的摩擦系数 -->
-            <mu2 value="20.0" />
-            <!-- 提高了摩擦力的配置，减小了刚度系数的配置,轮子是橡胶的，刚度没那么大 -->
-            <!-- 接触的刚度系数 -->
-            <kp value="1000000000.0" />
-            <!-- 阻尼系数 -->
-            <kd value="1.0" />
-        </gazebo>
-    </xacro:macro>
-    <!-- 6.调用宏生成多个车轮 -->
-    <xacro:wheel_func link_name="front_left" front_flag="1" left_flag="1" />
-    <xacro:wheel_func link_name="front_right" front_flag="1" left_flag="-1" />
-    <!-- <xacro:wheel_func link_name="back_left" front_flag="-1" left_flag="1" /> -->
-    <!-- <xacro:wheel_func link_name="back_right" front_flag="-1" left_flag="-1" /> -->
-</robot>
+/home/wz/Desktop/ROS_ROBOT/src/cpp06_urdf/urdf/xacro/car_base.urdf.xacro

File: install/cpp06_urdf/share/cpp06_urdf/urdf/xacro/car_camera.urdf.xacro (robot description, xacro)
@@ -1,43 +1 @@
-<?xml version="1.0"?>
-<robot xmlns:xacro="http://www.ros.org/wiki/xacro">
-    <xacro:include filename="$(find cpp06_urdf)/urdf/xacro/common_inertia.xacro"/>
-    <!-- 声明一些参数 -->
-    <!-- 摄像头的长宽高 -->
-    <xacro:property name="PI" value="3.1415927" />
-    <xacro:property name="camera_x" value="0.01" />
-    <xacro:property name="camera_y" value="0.08" />
-    <xacro:property name="camera_z" value="0.01" />
-    <!-- 关节的偏移量 -->
-    <xacro:property name="camera_joint_x" value="${car_length/2 - 0.01}" />
-    <xacro:property name="camera_joint_y" value="0" />
-    <xacro:property name="camera_joint_z" value="${car_height / 2 + camera_z / 2}" />
-    <!-- 设置link和joint -->
-    <link name="camera">
-        <visual>
-            <geometry>
-                <box size="${camera_x} ${camera_y} ${camera_z}"/>
-            </geometry>
-        </visual>
-        <collision>
-            <geometry>
-                <box size="${camera_x} ${camera_y} ${camera_z}"/>
-            </geometry>
-        </collision>
-        <xacro:box_inertia m="1.0" d="${camera_x}" w="${camera_y}" h="${camera_z}" />
-    </link>
-    <link name="camera_optical_link">
-    </link>
-    <joint name="camera_optical_link2camera" type="fixed">
-        <parent link="camera"/>
-        <child link="camera_optical_link"/>
-        <origin xyz="0.0 0.0 0.0" rpy="${-PI/2} 0.0 ${-PI/2}"/>
-    </joint>
-    <joint name="camera2base_link" type="fixed">
-        <parent link="base_link"/>
-        <child link="camera"/>
-        <origin xyz="${camera_joint_x} ${camera_joint_y} ${camera_joint_z} "/>
-    </joint>
-    <gazebo reference="camera">
-        <material>Gazebo/Black</material>
-    </gazebo>
-</robot>
+/home/wz/Desktop/ROS_ROBOT/src/cpp06_urdf/urdf/xacro/car_camera.urdf.xacro

File: install/cpp06_urdf/share/cpp06_urdf/urdf/xacro/car_caster.urdf.xacro (robot description, xacro)
@@ -1,35 +1 @@
-<?xml version="1.0"?>
-<robot xmlns:xacro="http://www.ros.org/wiki/xacro">
-   <xacro:include filename="$(find cpp06_urdf)/urdf/xacro/common_inertia.xacro"/>
-    <xacro:property name="PI" value="3.1415927" />
-    <xacro:property name="caster_radius" value="0.01" />
-    <!-- 关节的偏移量 -->
-    <xacro:property name="caster_joint_x" value="-0.08" />
-    <xacro:property name="caster_joint_y" value="0" />
-    <xacro:property name="caster_joint_z" value="${-(car_height / 2 + distance - caster_radius)}" />
-    <!-- 设置link和joint -->
-    <link name="caster">
-        <visual>
-            <geometry>
-                <sphere radius="${caster_radius}"/>
-            </geometry>
-        </visual>
-        <collision>
-            <geometry>
-                <sphere radius="${caster_radius}"/>
-            </geometry>
-        </collision>
-        <xacro:sphere_inertia m="0.01" r="${caster_radius}" />
-    </link>
-    <joint name="caster2base_link" type="fixed">
-        <parent link="base_link"/>
-        <child link="caster"/>
-        <origin xyz="${caster_joint_x} ${caster_joint_y} ${caster_joint_z} "/>
-    </joint>
-    <gazebo reference="caster">
-        <mu1 value="0.0" />
-        <mu2 value="0.0" />
-        <kp value="1000000000.0" />
-        <kd value="1.0" />
-    </gazebo>
-</robot>
+/home/wz/Desktop/ROS_ROBOT/src/cpp06_urdf/urdf/xacro/car_caster.urdf.xacro

File: install/cpp06_urdf/share/cpp06_urdf/urdf/xacro/car_control.urdf.xacro (robot description, xacro)
@@ -1,46 +1 @@
-<?xml version="1.0"?>
-<robot xmlns:xacro="http://www.ros.org/wiki/xacro">
-    <xacro:macro name="car_control">
-    <ros2_control name="FishBotGazeboSystem" type="system">
-            <hardware>
-                <plugin>gazebo_ros2_control/GazeboSystem</plugin>
-            </hardware>
-            <joint name="front_left2base_link">
-                <command_interface name="velocity">
-                    <param name="min">-1</param>
-                    <param name="max">1</param>
-                </command_interface>
-                <command_interface name="effort">
-                    <param name="min">-0.1</param>
-                    <param name="max">0.1</param>
-                </command_interface>
-                <state_interface name="position" />
-                <state_interface name="velocity" />
-                <state_interface name="effort" />
-            </joint>
-            <joint name="front_right2base_link">
-                <command_interface name="velocity">
-                    <param name="min">-1</param>
-                    <param name="max">1</param>
-                </command_interface>
-                <command_interface name="effort">
-                    <param name="min">-0.1</param>
-                    <param name="max">0.1</param>
-                </command_interface>
-                <state_interface name="position" />
-                <state_interface name="velocity" />
-                <state_interface name="effort" />
-            </joint>
-        </ros2_control>
-        <gazebo>
-        <plugin filename="libgazebo_ros2_control.so" name="gazebo_ros2_control">
-            <parameters>$(find cpp06_urdf)/config/car_controller.yaml</parameters>
-            <!-- 话题的重映射 -->
-            <ros>
-                <remapping>/car_diff_drive_controller/cmd_vel_unstamped:=/cmd_vel</remapping>
-                <remapping>/car_diff_drive_controller/odom:=/odom</remapping>
-            </ros>
-        </plugin>
-</gazebo>
-    </xacro:macro>
-</robot>
+/home/wz/Desktop/ROS_ROBOT/src/cpp06_urdf/urdf/xacro/car_control.urdf.xacro

File: install/cpp06_urdf/share/cpp06_urdf/urdf/xacro/car_imu.urdf.xacro (robot description, xacro)
@@ -1,32 +1 @@
-<?xml version="1.0"?>
-<robot xmlns:xacro="http://www.ros.org/wiki/xacro">
-   <xacro:include filename="$(find cpp06_urdf)/urdf/xacro/common_inertia.xacro"/>
-    <xacro:macro name="imu_xacro" params="xyz">
-        <link name="imu">
-            <visual>
-                <origin xyz="0 0 0" rpy="0 0 0" />
-                <geometry>
-                    <box size="0.02 0.02 0.02" />
-                </geometry>
-                <material name="black">
-                    <color rgba="0 0 0 0.8" />
-                </material>
-            </visual>
-            <collision>
-                <origin xyz="0 0 0" rpy="0 0 0" />
-                <geometry>
-                    <box size="0.02 0.02 0.02" />
-                </geometry>
-                <material name="black">
-                    <color rgba="0 0 0 0.8" />
-                </material>
-            </collision>
-            <xacro:box_inertia m="0.01" w="0.02" d="0.02" h="0.02"/>
-        </link>
-        <joint name="imu2base_link" type="fixed">
-            <parent link="base_link" />
-            <child link="imu" />
-            <origin xyz="${xyz}" />
-        </joint>
-    </xacro:macro>
-</robot>
+/home/wz/Desktop/ROS_ROBOT/src/cpp06_urdf/urdf/xacro/car_imu.urdf.xacro

File: install/cpp06_urdf/share/cpp06_urdf/urdf/xacro/car_laser.urdf.xacro (robot description, xacro)
@@ -1,40 +1 @@
-<?xml version="1.0"?>
-<robot xmlns:xacro="http://www.ros.org/wiki/xacro">
-    <xacro:include filename="$(find cpp06_urdf)/urdf/xacro/common_inertia.xacro"/>
-    <!-- 声明变量 -->
-    <!-- 雷达尺寸 -->
-    <xacro:property name="laser_radius" value="0.03" />
-    <xacro:property name="laser_length" value="0.03" />
-    <!-- 雷达关节偏移量 -->
-    <xacro:property name="laser_joint_x" value="0" />
-    <xacro:property name="laser_joint_y" value="0" />
-    <xacro:property name="laser_joint_z" value="${car_height / 2 + laser_length / 2}" />
-    <!-- 设置link和joint -->
-    <link name="laser">
-        <visual>
-            <geometry>
-                <cylinder radius="${laser_radius}" length="${laser_length}"/>
-            </geometry>
-            <material name="blue">
-                <color rgba="0.1 0.1 0.7 0.8"/>
-            </material>
-        </visual>
-        <collision>
-            <geometry>
-                <cylinder radius="${laser_radius}" length="${laser_length}"/>
-            </geometry>
-            <material name="blue">
-                <color rgba="0.1 0.1 0.7 0.8"/>
-            </material>
-        </collision>
-        <xacro:cylinder_inertia m="1.0" r="${laser_radius}" h="${laser_length}" />
-    </link>
-    <joint name="laser2base_link" type="fixed">
-        <parent link="base_link"/>
-        <child link="laser"/>
-        <origin xyz="${laser_joint_x} ${laser_joint_y} ${laser_joint_z}"/>
-    </joint>
-    <gazebo reference="laser">
-        <material>Gazebo/Black</material>
-    </gazebo>
-</robot>
+/home/wz/Desktop/ROS_ROBOT/src/cpp06_urdf/urdf/xacro/car_laser.urdf.xacro

File: install/cpp06_urdf/share/cpp06_urdf/urdf/xacro/common_inertia.xacro (robot description, xacro)
@@ -1,21 +1 @@
-<?xml version="1.0"?>
-<robot xmlns:xacro="http://ros.org/wiki/xacro">
-    <xacro:macro name="box_inertia" params="m w h d">
-        <inertial>
-            <mass value="${m}" />
-            <inertia ixx="${(m/12) * (h*h + d*d)}" ixy="0.0" ixz="0.0" iyy="${(m/12) * (w*w + d*d)}" iyz="0.0" izz="${(m/12) * (w*w + h*h)}" />
-        </inertial>
-    </xacro:macro>
-    <xacro:macro name="cylinder_inertia" params="m r h">
-        <inertial>
-            <mass value="${m}" />
-            <inertia ixx="${(m/12) * (3*r*r + h*h)}" ixy="0" ixz="0" iyy="${(m/12) * (3*r*r + h*h)}" iyz="0" izz="${(m/2) * (r*r)}" />
-        </inertial>
-    </xacro:macro>
-    <xacro:macro name="sphere_inertia" params="m r">
-        <inertial>
-            <mass value="${m}" />
-            <inertia ixx="${(2/5) * m * (r*r)}" ixy="0.0" ixz="0.0" iyy="${(2/5) * m * (r*r)}" iyz="0.0" izz="${(2/5) * m * (r*r)}" />
-        </inertial>
-    </xacro:macro>
-</robot>
+/home/wz/Desktop/ROS_ROBOT/src/cpp06_urdf/urdf/xacro/common_inertia.xacro

File: install/cpp06_urdf/share/cpp06_urdf/urdf/xacro/demo01_helloworld.urdf.xacro (robot description, xacro)
@@ -1,27 +1 @@
-<?xml version="1.0"?>
-<robot name="my_car" xmlns:xacro="http://wiki.ros.org/xacro">
-  <!-- 参数定义 -->
-  <xacro:property name="wheel_radius" value="0.025" />
-  <xacro:property name="wheel_length" value="0.02" />
-  <xacro:property name="PI" value="3.1415927" />
-  <!-- 轮子宏定义 -->
-  <xacro:macro name="wheel_func" params="wheel_name">
-    <link name="${wheel_name}_wheel">
-      <visual>
-        <geometry>
-          <!-- 修正：使用预定义属性而非宏参数 -->
-          <cylinder radius="${wheel_radius}" length="${wheel_length}"/>
-        </geometry>
-        <origin xyz="0 0 0" rpy="${PI/2} 0 0"/>
-        <material name="wheel_color">
-          <color rgba="0 0 0 0.3"/>
-        </material>
-      </visual>
-    </link>
-  </xacro:macro>
-  <!-- 宏调用 -->
-  <xacro:wheel_func wheel_name="left_front"/>
-  <xacro:wheel_func wheel_name="left_back"/>
-  <xacro:wheel_func wheel_name="right_front"/>
-  <xacro:wheel_func wheel_name="right_back"/>
-</robot>
+/home/wz/Desktop/ROS_ROBOT/src/cpp06_urdf/urdf/xacro/demo01_helloworld.urdf.xacro

File: install/cpp06_urdf/share/cpp06_urdf/urdf/xacro/demo02_base_pro.urdf.xacro (robot description, xacro)
@@ -1,14 +1 @@
-<!--
-1. 变量定义（声明）
-2. 变量调用
-3. 变量运算
--->
-<robot xmlns:xacro="http://www.ros.org/wiki/xacro" name="demo02_pro">
-    <!-- 1. 变量定义（声明） -->
-    <xacro:property name="num1" value="10" />
-    <xacro:property name="num2" value="20" />
-    <!-- 2. 变量调用 -->
-    <car length="${num1}" width="${num2}" />
-    <!-- 3. 变量运算 -->
-    <sum value="${num1 + num2}" />
-</robot>
+/home/wz/Desktop/ROS_ROBOT/src/cpp06_urdf/urdf/xacro/demo02_base_pro.urdf.xacro

File: install/cpp06_urdf/share/cpp06_urdf/urdf/xacro/demo03_base_func.urdf.xacro (robot description, xacro)
@@ -1,10 +1 @@
-<!-- 演示宏的定义和调用 -->
-<robot xmlns:xacro="http://www.ros.org/wiki/xacro" name="demo03_func">
-    <!-- 宏定义 -->
-    <xacro:macro name="get_sum" params="num1 num2">
-        <sum value="${num1 + num2}" />
-    </xacro:macro>
-    <!-- 宏调用 -->
-    <xacro:get_sum num1="20" num2="30" />
-    <xacro:get_sum num1="70" num2="30" />
-</robot>
+/home/wz/Desktop/ROS_ROBOT/src/cpp06_urdf/urdf/xacro/demo03_base_func.urdf.xacro

File: install/cpp06_urdf/share/cpp06_urdf/urdf/xacro/demo04_base_include.urdf.xacro (robot description, xacro)
@@ -1,5 +1 @@
-<!-- 需求：包含其他xacro文件 -->
-<robot xmlns:xacro="http://www.ros.org/wiki/xacro" name="demo04_include">
-    <xacro:include filename="demo02_base_pro.urdf.xacro" />
-    <xacro:include filename="demo03_base_func.urdf.xacro" />
-</robot>
+/home/wz/Desktop/ROS_ROBOT/src/cpp06_urdf/urdf/xacro/demo04_base_include.urdf.xacro

File: install/cpp06_urdf/share/cpp06_urdf/urdf/xacro/gazebo_control_plugin.xacro (robot description, xacro)
@@ -1,30 +1 @@
-<?xml version="1.0"?>
-<robot xmlns:xacro="http://www.ros.org/wiki/xacro">
-    <xacro:macro name="gazebo_control_plugin">
-        <gazebo>
-            <plugin name='diff_drive' filename='libgazebo_ros_diff_drive.so'>
-                <ros>
-                    <namespace>/</namespace>
-                    <remapping>cmd_vel:=cmd_vel</remapping>
-                    <remapping>odom:=odom</remapping>
-                </ros>
-                <update_rate>30</update_rate>
-                <!-- wheels -->
-                <left_joint>front_left2base_link</left_joint>
-                <right_joint>front_right2base_link</right_joint>
-                <!-- kinematics -->
-                <wheel_separation>0.2</wheel_separation>
-                <wheel_diameter>0.064</wheel_diameter>
-                <!-- limits -->
-                <max_wheel_torque>20</max_wheel_torque>
-                <max_wheel_acceleration>1.0</max_wheel_acceleration>
-                <!-- output -->
-                <publish_odom>true</publish_odom>
-                <publish_odom_tf>true</publish_odom_tf>
-                <publish_wheel_tf>true</publish_wheel_tf>
-                <odometry_frame>odom</odometry_frame>
-                <robot_base_frame>base_footprint</robot_base_frame>
-            </plugin>
-        </gazebo>
-   </xacro:macro>
-</robot>
+/home/wz/Desktop/ROS_ROBOT/src/cpp06_urdf/urdf/xacro/gazebo_control_plugin.xacro
