Commit message: Perfected readme,Python invoked the MoveIt inverse kinematics interface.

File: install/cpp06_urdf/share/cpp06_urdf/urdf/xacro/gazebo_sensor_plugin.xacro (robot description, xacro)
@@ -1,138 +1 @@
-<?xml version="1.0"?>
-<robot xmlns:xacro="http://www.ros.org/wiki/xacro">
-    <xacro:macro name="gazebo_sensor_plugin">
-        <gazebo reference="laser">
-            <sensor name="laserscan" type="ray">
-                <plugin name="laserscan" filename="libgazebo_ros_ray_sensor.so">
-                    <ros>
-                        <namespace>/</namespace>
-                        <remapping>~/out:=scan</remapping>
-                    </ros>
-                    <output_type>sensor_msgs/LaserScan</output_type>
-                    <frame_name>laser</frame_name>
-                </plugin>
-                <always_on>true</always_on>
-                <visualize>true</visualize>
-                <update_rate>5</update_rate>
-                <pose>0 0 0 0 0 0</pose>
-				<!-- 激光传感器配置 -->
-                <ray>
-                    <!-- 设置扫描范围 -->
-                    <scan>
-                        <horizontal>
-                            <samples>360</samples>
-                            <resolution>1.000000</resolution>
-                            <min_angle>0.000000</min_angle>
-                            <max_angle>6.280000</max_angle>
-                        </horizontal>
-                    </scan>
-                    <!-- 设置扫描距离 -->
-                    <range>
-                        <min>0.120000</min>
-                        <max>8.0</max>
-                        <resolution>0.015000</resolution>
-                    </range>
-                    <!-- 设置噪声 -->
-                    <noise>
-                        <type>gaussian</type>
-                        <mean>0.0</mean>
-                        <stddev>0.01</stddev>
-                    </noise>
-                </ray>
-            </sensor>
-        </gazebo>
-<gazebo reference="imu">
-    <sensor name="imu_sensor" type="imu">
-        <plugin name="imu_plugin" filename="libgazebo_ros_imu_sensor.so">
-            <ros>
-                <namespace>/</namespace>
-                <remapping>~/out:=imu</remapping>
-            </ros>
-            <initial_orientation_as_reference>false</initial_orientation_as_reference>
-        </plugin>
-        <update_rate>100</update_rate>
-        <always_on>true</always_on>
-        <!-- 六轴噪声设置 -->
-        <imu>
-            <angular_velocity>
-                <x>
-                    <noise type="gaussian">
-                        <mean>0.0</mean>
-                        <stddev>2e-4</stddev>
-                        <bias_mean>0.0000075</bias_mean>
-                        <bias_stddev>0.0000008</bias_stddev>
-                    </noise>
-                </x>
-                <y>
-                    <noise type="gaussian">
-                        <mean>0.0</mean>
-                        <stddev>2e-4</stddev>
-                        <bias_mean>0.0000075</bias_mean>
-                        <bias_stddev>0.0000008</bias_stddev>
-                    </noise>
-                </y>
-                <z>
-                    <noise type="gaussian">
-                        <mean>0.0</mean>
-                        <stddev>2e-4</stddev>
-                        <bias_mean>0.0000075</bias_mean>
-                        <bias_stddev>0.0000008</bias_stddev>
-                    </noise>
-                </z>
-            </angular_velocity>
-            <linear_acceleration>
-                <x>
-                    <noise type="gaussian">
-                        <mean>0.0</mean>
-                        <stddev>1.7e-2</stddev>
-                        <bias_mean>0.1</bias_mean>
-                        <bias_stddev>0.001</bias_stddev>
-                    </noise>
-                </x>
-                <y>
-                    <noise type="gaussian">
-                        <mean>0.0</mean>
-                        <stddev>1.7e-2</stddev>
-                        <bias_mean>0.1</bias_mean>
-                        <bias_stddev>0.001</bias_stddev>
-                    </noise>
-                </y>
-                <z>
-                    <noise type="gaussian">
-                        <mean>0.0</mean>
-                        <stddev>1.7e-2</stddev>
-                        <bias_mean>0.1</bias_mean>
-                        <bias_stddev>0.001</bias_stddev>
-                    </noise>
-                </z>
-            </linear_acceleration>
-        </imu>
-    </sensor>
-</gazebo>
-    </xacro:macro>
-<gazebo reference="camera">
-    <sensor type="depth" name="camera_sensor">
-        <plugin name="depth_camera" filename="libgazebo_ros_camera.so">
-            <frame_name>camera_optical_link</frame_name>
-        </plugin>
-        <always_on>true</always_on>
-        <update_rate>10</update_rate>
-        <camera name="camera">
-            <horizontal_fov>1.5009831567</horizontal_fov>
-            <image>
-                <width>800</width>
-                <height>600</height>
-                <format>R8G8B8</format>
-            </image>
-            <distortion>
-                <k1>0.0</k1>
-                <k2>0.0</k2>
-                <k3>0.0</k3>
-                <p1>0.0</p1>
-                <p2>0.0</p2>
-                <center>0.5 0.5</center>
-            </distortion>
-        </camera>
-    </sensor>
-</gazebo>
-</robot>
+/home/wz/Desktop/ROS_ROBOT/src/cpp06_urdf/urdf/xacro/gazebo_sensor_plugin.xacro

File: install/cpp06_urdf/share/cpp06_urdf/urdf/xacro/robot_description.urdf.xacro (robot description, xacro)
@@ -1,375 +1 @@
-<?xml version="1.0" ?>
-<robot name="NanoRobot"  xmlns:xacro="http://ros.org/wiki/xacro">
-  <xacro:arg name="robot_name" default=""/>
-  <xacro:include filename="$(find cpp06_urdf)/urdf/urdf/robot_description.gazebo.xacro" />
-  <link name="$(arg robot_name)/base_footprint"/>
-  <joint name="base_joint" type="fixed">
-    <parent link="$(arg robot_name)/base_footprint"/>
-    <child link="$(arg robot_name)/base_link"/>
-    <origin xyz="0.0 0.0 0.012" rpy="0 0 3.1415926"/>
-  </joint>
-  <link
-    name="$(arg robot_name)/base_link">
-    <inertial>
-      <origin
-        xyz="-0.021363490239433 0.000185677952833835 0.0417013760059846"
-        rpy="0 0 0" />
-      <mass
-        value="0.1" />
-      <inertia
-        ixx="0.00169347433894092"
-        ixy="-2.48653191534453E-07"
-        ixz="3.6777445179091E-05"
-        iyy="0.00104562302644335"
-        iyz="-4.01932028426777E-06"
-        izz="0.00148226749250531" />
-    </inertial>
-    <visual>
-      <origin
-        xyz="0 0 0"
-        rpy="0 0 0" />
-      <geometry>
-        <mesh
-          filename="package://cpp06_urdf/meshes/base_link.STL" />
-      </geometry>
-      <material
-        name="">
-        <color
-          rgba="1 1 1 1" />
-      </material>
-    </visual>
-    <collision>
-      <origin
-        xyz="0 0 0"
-        rpy="0 0 0" />
-      <geometry>
-        <mesh
-          filename="package://cpp06_urdf/meshes/base_link.STL" />
-      </geometry>
-    </collision>
-  </link>
-  <link
-    name="$(arg robot_name)/imu">
-    <inertial>
-      <origin
-        xyz="3.46944695195361E-18 0 -0.00353385896202057"
-        rpy="0 0 0" />
-      <mass
-        value="0.000834" />
-      <inertia
-        ixx="1.72751258992806E-08"
-        ixy="2.49134059713724E-24"
-        ixz="-2.52435489670724E-26"
-        iyy="1.01251258992806E-08"
-        iyz="1.8466691376894E-25"
-        izz="2.3801E-08" />
-    </inertial>
-    <visual>
-      <origin
-        xyz="0 0 0"
-        rpy="0 0 0" />
-      <geometry>
-        <mesh
-          filename="package://cpp06_urdf/meshes/imu.STL" />
-      </geometry>
-      <material
-        name="">
-        <color
-          rgba="1 1 1 1" />
-      </material>
-    </visual>
-    <collision>
-      <origin
-        xyz="0 0 0"
-        rpy="0 0 0" />
-      <geometry>
-        <mesh
-          filename="package://cpp06_urdf/meshes/imu.STL" />
-      </geometry>
-    </collision>
-  </link>
-  <joint
-    name="imu_joint"
-    type="fixed">
-    <origin
-      xyz="-0.056956 -0.0059543 0.072756"
-      rpy="0 5.2369E-16 0" />
-    <parent
-      link="$(arg robot_name)/base_link" />
-    <child
-      link="$(arg robot_name)/imu" />
-    <axis
-      xyz="0 0 0" />
-  </joint>
-  <link
-    name="$(arg robot_name)/base_camera_link">
-    <inertial>
-      <origin
-        xyz="-0.0045346942299942 1.38777878078145E-17 -0.00179125965737512"
-        rpy="0 0 0" />
-      <mass
-        value="0.00100487943921971" />
-      <inertia
-        ixx="7.55677391275611E-08"
-        ixy="-2.39038796583022E-24"
-        ixz="-1.37755038601046E-09"
-        iyy="3.94938932151791E-08"
-        iyz="2.43323642233816E-23"
-        izz="4.01523294449251E-08" />
-    </inertial>
-    <visual>
-      <origin
-        xyz="0 0 0"
-        rpy="0 0 0" />
-      <geometry>
-        <mesh
-          filename="package://cpp06_urdf/meshes/base_camera_link.STL" />
-      </geometry>
-      <material
-        name="">
-        <color
-          rgba="1 1 1 1" />
-      </material>
-    </visual>
-    <collision>
-      <origin
-        xyz="0 0 0"
-        rpy="0 0 0" />
-      <geometry>
-        <mesh
-          filename="package://cpp06_urdf/meshes/base_camera_link.STL" />
-      </geometry>
-    </collision>
-  </link>
-  <joint
-    name="camera_joint"
-    type="fixed">
-    <origin
-      xyz="0.0277 0 0.0623"
-      rpy="-2.2337E-16 0.2 0" />
-    <parent
-      link="$(arg robot_name)/base_link" />
-    <child
-      link="$(arg robot_name)/base_camera_link" />
-    <axis
-      xyz="0 0 0" />
-  </joint>
-  <link
-    name="$(arg robot_name)/base_laser_link">
-    <inertial>
-      <origin
-        xyz="-0.00911214120076251 0.000185677952834168 -0.0842986239940154"
-        rpy="0 0 0" />
-      <mass
-        value="0.1" />
-      <inertia
-        ixx="0.00169347433894092"
-        ixy="-2.4865319153732E-07"
-        ixz="3.67774451790908E-05"
-        iyy="0.00104562302644335"
-        iyz="-4.01932028426874E-06"
-        izz="0.00148226749250531" />
-    </inertial>
-    <visual>
-      <origin
-        xyz="0 0 0"
-        rpy="0 0 0" />
-      <geometry>
-        <mesh
-          filename="package://cpp06_urdf/meshes/base_laser_link.STL" />
-      </geometry>
-      <material
-        name="">
-        <color
-          rgba="1 1 1 1" />
-      </material>
-    </visual>
-    <collision>
-      <origin
-        xyz="0 0 0"
-        rpy="0 0 0" />
-      <geometry>
-        <mesh
-          filename="package://cpp06_urdf/meshes/base_laser_link.STL" />
-      </geometry>
-    </collision>
-  </link>
-  <joint
-    name="laser_joint"
-    type="fixed">
-    <origin
-      xyz="-0.012251 0 0.126"
-      rpy="-1.6843E-15 -1.0776E-15 4.3793E-15" />
-    <parent
-      link="$(arg robot_name)/base_link" />
-    <child
-      link="$(arg robot_name)/base_laser_link" />
-    <axis
-      xyz="0 0 0" />
-  </joint>
-  <link
-    name="$(arg robot_name)/left_wheel_link">
-    <inertial>
-      <origin
-        xyz="-6.93889390390723E-18 3.46944695195361E-18 0.017494370940819"
-        rpy="0 0 0" />
-      <mass
-        value="0.0561341413751443" />
-      <inertia
-        ixx="2.45284373382495E-05"
-        ixy="1.79487710154599E-21"
-        ixz="7.36303183829231E-18"
-        iyy="2.45284373382495E-05"
-        iyz="1.73397416098309E-17"
-        izz="4.23355136524843E-05" />
-    </inertial>
-    <visual>
-      <origin
-        xyz="0 0 0"
-        rpy="0 0 0" />
-      <geometry>
-        <mesh
-          filename="package://cpp06_urdf/meshes/left_wheel_link.STL" />
-      </geometry>
-      <material
-        name="">
-        <color
-          rgba="0.109803921568627 0.109803921568627 0.109803921568627 1" />
-      </material>
-    </visual>
-    <collision>
-      <origin
-        xyz="0 0 0"
-        rpy="0 0 0" />
-      <geometry>
-        <mesh
-          filename="package://cpp06_urdf/meshes/left_wheel_link.STL" />
-      </geometry>
-    </collision>
-  </link>
-  <joint
-    name="left_wheel_joint"
-    type="continuous">
-    <origin
-      xyz="0 0.0658 0.02275"
-      rpy="-1.5708 5.2369E-16 8.6736E-17" />
-    <parent
-      link="$(arg robot_name)/base_link" />
-    <child
-      link="$(arg robot_name)/left_wheel_link" />
-    <axis
-      xyz="0 0 1" />
-    <limit
-      effort="100"
-      velocity="100" />
-  </joint>
-  <link
-    name="$(arg robot_name)/right_wheel_link">
-    <inertial>
-      <origin
-        xyz="3.46944695195361E-18 -1.73472347597681E-18 -0.017494370940819"
-        rpy="0 0 0" />
-      <mass
-        value="0.0561341413751443" />
-      <inertia
-        ixx="2.45284373382495E-05"
-        ixy="-1.10855737450343E-21"
-        ixz="-7.37237567686968E-18"
-        iyy="2.45284373382495E-05"
-        iyz="1.734064769358E-17"
-        izz="4.23355136524843E-05" />
-    </inertial>
-    <visual>
-      <origin
-        xyz="0 0 0"
-        rpy="0 0 0" />
-      <geometry>
-        <mesh
-          filename="package://cpp06_urdf/meshes/right_wheel_link.STL" />
-      </geometry>
-      <material
-        name="">
-        <color
-          rgba="0.109803921568627 0.109803921568627 0.109803921568627 1" />
-      </material>
-    </visual>
-    <collision>
-      <origin
-        xyz="0 0 0"
-        rpy="0 0 0" />
-      <geometry>
-        <mesh
-          filename="package://cpp06_urdf/meshes/right_wheel_link.STL" />
-      </geometry>
-    </collision>
-  </link>
-  <joint
-    name="right_wheel_joint"
-    type="continuous">
-    <origin
-      xyz="0 -0.0658 0.02275"
-      rpy="1.5708 -5.2369E-16 3.1416" />
-    <parent
-      link="$(arg robot_name)/base_link" />
-    <child
-      link="$(arg robot_name)/right_wheel_link" />
-    <axis
-      xyz="0 0 1" />
-    <limit
-      effort="100"
-      velocity="100" />
-  </joint>
-  <link
-    name="$(arg robot_name)/ball_wheel_link">
-    <inertial>
-      <origin
-        xyz="-0.00805 0 0"
-        rpy="0 0 0" />
-      <mass
-        value="0.00218512482182764" />
-      <inertia
-        ixx="5.66406205065944E-08"
-        ixy="0"
-        ixz="0"
-        iyy="5.66406205065944E-08"
-        iyz="0"
-        izz="5.66406205065944E-08" />
-    </inertial>
-    <visual>
-      <origin
-        xyz="0 0 0"
-        rpy="0 0 0" />
-      <geometry>
-        <mesh
-          filename="package://cpp06_urdf/meshes/ball_wheel_link.STL" />
-      </geometry>
-      <material
-        name="">
-        <color
-          rgba="1 1 1 1" />
-      </material>
-    </visual>
-    <collision>
-      <origin
-        xyz="0 0 0"
-        rpy="0 0 0" />
-      <geometry>
-        <mesh
-          filename="package://cpp06_urdf/meshes/ball_wheel_link.STL" />
-      </geometry>
-    </collision>
-  </link>
-  <joint
-    name="ball_wheel_joint"
-    type="fixed">
-    <origin
-      xyz="-0.06445 0 -0.0028"
-      rpy="0 5.2369E-16 0" />
-    <parent
-      link="$(arg robot_name)/base_link" />
-    <child
-      link="$(arg robot_name)/ball_wheel_link" />
-    <axis
-      xyz="0 0 0" />
-  </joint>
-</robot>
+/home/wz/Desktop/ROS_ROBOT/src/cpp06_urdf/urdf/xacro/robot_description.urdf.xacro

File: install/test_moveit_config/share/test_moveit_config/config/arm_BRTIRUS0805A_SLDASM.ros2_control.xacro (robot description, xacro)
@@ -1,60 +1 @@
-<?xml version="1.0"?>
-<robot xmlns:xacro="http://www.ros.org/wiki/xacro">
-    <xacro:macro name="arm_BRTIRUS0805A_SLDASM_ros2_control" params="name initial_positions_file">
-        <xacro:property name="initial_positions" value="${load_yaml(initial_positions_file)['initial_positions']}"/>
-        <ros2_control name="${name}" type="system">
-            <hardware>
-                <!-- By default, set up controllers for simulation. This won't work on real hardware -->
-                <plugin>mock_components/GenericSystem</plugin>
-            </hardware>
-            <joint name="joint1">
-                <command_interface name="position"/>
-                <command_interface name="velocity"/>
-                <state_interface name="position">
-                  <param name="initial_value">${initial_positions['joint1']}</param>
-                </state_interface>
-                <state_interface name="velocity"/>
-            </joint>
-            <joint name="joint2">
-                <command_interface name="position"/>
-                <command_interface name="velocity"/>
-                <state_interface name="position">
-                  <param name="initial_value">${initial_positions['joint2']}</param>
-                </state_interface>
-                <state_interface name="velocity"/>
-            </joint>
-            <joint name="joint3">
-                <command_interface name="position"/>
-                <command_interface name="velocity"/>
-                <state_interface name="position">
-                  <param name="initial_value">${initial_positions['joint3']}</param>
-                </state_interface>
-                <state_interface name="velocity"/>
-            </joint>
-            <joint name="joint4">
-                <command_interface name="position"/>
-                <command_interface name="velocity"/>
-                <state_interface name="position">
-                  <param name="initial_value">${initial_positions['joint4']}</param>
-                </state_interface>
-                <state_interface name="velocity"/>
-            </joint>
-            <joint name="joint5">
-                <command_interface name="position"/>
-                <command_interface name="velocity"/>
-                <state_interface name="position">
-                  <param name="initial_value">${initial_positions['joint5']}</param>
-                </state_interface>
-                <state_interface name="velocity"/>
-            </joint>
-            <joint name="joint6">
-                <command_interface name="position"/>
-                <command_interface name="velocity"/>
-                <state_interface name="position">
-                  <param name="initial_value">${initial_positions['joint6']}</param>
-                </state_interface>
-                <state_interface name="velocity"/>
-            </joint>
-        </ros2_control>
-    </xacro:macro>
-</robot>
+/home/wz/Desktop/ROS_ROBOT/src/test_moveit_config/config/arm_BRTIRUS0805A_SLDASM.ros2_control.xacro

File: install/test_moveit_config/share/test_moveit_config/config/arm_BRTIRUS0805A_SLDASM.urdf.xacro (robot description, xacro)
@@ -1,9 +1 @@
-<?xml version="1.0"?>
-<robot xmlns:xacro="http://www.ros.org/wiki/xacro" name="arm_BRTIRUS0805A_SLDASM">
-    <xacro:arg name="initial_positions_file" default="initial_positions.yaml" />
-    <!-- Import arm_BRTIRUS0805A_SLDASM urdf file -->
-    <xacro:include filename="$(find cpp06_urdf)/urdf/urdf/arm_BRTIRUS0805A_SLDASM.urdf" />
-    <!-- Import control_xacro -->
-    <xacro:include filename="arm_BRTIRUS0805A_SLDASM.ros2_control.xacro" />
-    <xacro:arm_BRTIRUS0805A_SLDASM_ros2_control name="FakeSystem" initial_positions_file="$(arg initial_positions_file)"/>
-</robot>
+/home/wz/Desktop/ROS_ROBOT/src/test_moveit_config/config/arm_BRTIRUS0805A_SLDASM.urdf.xacro
